File: kicad_convert/kicad_sch/NPN1.kicad_sch (KiCad schematic)
At the start: 6 parts, among them Q1 NPN

Commit message: save
Connections:
- net V1 renamed 12
Changed lines of the file:
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@@
 			)
 		)
-		(property "Value" "V1"
+		(property "Value" "12"
 			(at 95.25 77.47 0)
 			(show_name no)
